File: ASAM_Schematic_Updated/SAM.kicad_sch (KiCad schematic)
At the start: 37 parts, among them M18 Battery-18V, P1 Potentiometer, U1 ATmega2560-16A, U2 ADS1115, U3 MAX6126 - Voltage Regulator, U4 PSI Sensor, U5 LCD

Commit message: updated schematic
Connections:
- net GND: no longer B1.1, B2.1
- new net 3V: B1.1, B2.1
Changed lines of the file:
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@@
+    (stroke (width 0) (type default) (color 0 0 0 0))
+  )
+  (wire (pts (xy 87.63 290.83) (xy 90.17 290.83))
     (stroke (width 0) (type default) (color 0 0 0 0))
   )
@@
     (stroke (width 0) (type default) (color 0 0 0 1))
   )
-  (wire (pts (xy 83.82 302.26) (xy 83.82 303.53))
-    (stroke (width 0) (type default) (color 0 0 0 0))
-  )
   (wire (pts (xy 81.28 71.12) (xy 81.28 72.39))
     (stroke (width 0) (type default) (color 0 0 0 0))
@@
     (stroke (width 0) (type default) (color 0 0 0 0))
   )
-  (wire (pts (xy 85.09 290.83) (xy 85.09 292.1))
-    (stroke (width 0) (type default) (color 0 0 0 0))
-  )
   (wire (pts (xy 78.74 222.25) (xy 86.36 222.25))
     (stroke (width 0) (type default) (color 0 0 0 0))
@@
   )
   (wire (pts (xy 226.06 160.02) (xy 226.06 158.75))
-    (stroke (width 0) (type default) (color 0 0 0 0))
-  )
-  (wire (pts (xy 83.82 302.26) (xy 90.17 302.26))
     (stroke (width 0) (type default) (color 0 0 0 0))
   )
@@
     (stroke (width 0) (type default) (color 0 0 0 1))
   )
-  (wire (pts (xy 85.09 290.83) (xy 90.17 290.83))
-    (stroke (width 0) (type default) (color 0 0 0 0))
-  )
   (bus (pts (xy 116.84 229.87) (xy 116.84 64.77))
     (stroke (width 0) (type default) (color 0 0 0 1))
@@
   )
   (wire (pts (xy 66.04 252.73) (xy 66.04 257.81))
+    (stroke (width 0) (type default) (color 0 0 0 0))
+  )
+  (wire (pts (xy 87.63 302.26) (xy 90.17 302.26))
     (stroke (width 0) (type default) (color 0 0 0 0))
   )
@@
     )
   )
+  (global_label "3V" (shape input) (at 87.63 302.26 180) (fields_autoplaced)
+    (effects (font (size 1.27 1.27) (thickness 0.254) bold) (justify right))
+    (property "Intersheet References" "${INTERSHEET_REFS}" (id 0) (at 82.7284 302.133 0)
+      (effects (font (size 1.27 1.27) (thickness 0.254) bold) (justify right) hide)
+    )
+  )
   (global_label "Linear Actuator (Right) -" (shape input) (at 227.33 292.1 180) (fields_autoplaced)
     (effects (font (size 1.27 1.27)) (justify right))
@@
     (property "Intersheet References" "${INTERSHEET_REFS}" (id 0) (at 250.0631 156.1306 0)
       (effects (font (size 1.27 1.27)) (justify left) hide)
+    )
+  )
+  (global_label "3V" (shape input) (at 87.63 290.83 180) (fields_autoplaced)
+    (effects (font (size 1.27 1.27) (thickness 0.254) bold) (justify right))
+    (property "Intersheet References" "${INTERSHEET_REFS}" (id 0) (at 82.7284 290.703 0)
+      (effects (font (size 1.27 1.27) (thickness 0.254) bold) (justify right) hide)
     )
   )
@@
     (pin "8")
   )
-  (symbol (lib_id "power:GND") (at 85.09 292.1 0) (unit 1)
-    (in_bom yes) (on_board yes)
-    (property "Reference" "#PWR?" (id 0) (at 85.09 298.45 0)
-      (effects (font (size 1.27 1.27)) hide)
-    )
-    (property "Value" "GND" (id 1) (at 85.09 295.91 0))
-    (property "Footprint" "" (id 2) (at 85.09 292.1 0)
-      (effects (font (size 1.27 1.27)) hide)
-    )
-    (property "Datasheet" "" (id 3) (at 85.09 292.1 0)
-      (effects (font (size 1.27 1.27)) hide)
-    )
-    (pin "1")
-  )
   (symbol (lib_id "Device:Battery") (at 175.26 80.01 0) (unit 1)
     (in_bom yes) (on_board yes) (fields_autoplaced)
@@
     (pin "1")
   )
-  (symbol (lib_id "power:GND") (at 83.82 303.53 0) (unit 1)
-    (in_bom yes) (on_board yes)
-    (property "Reference" "#PWR?" (id 0) (at 83.82 309.88 0)
-      (effects (font (size 1.27 1.27)) hide)
-    )
-    (property "Value" "GND" (id 1) (at 83.82 307.34 0))
-    (property "Footprint" "" (id 2) (at 83.82 303.53 0)
-      (effects (font (size 1.27 1.27)) hide)
-    )
-    (property "Datasheet" "" (id 3) (at 83.82 303.53 0)
-      (effects (font (size 1.27 1.27)) hide)
-    )
-    (pin "1")
-  )
   (symbol (lib_id "power:GND") (at 40.64 353.06 0) (unit 1)
     (in_bom yes) (on_board yes) (fields_autoplaced)
@@
       (reference "#PWR?") (unit 1) (value "GND") (footprint "")
     )
-    (path "/d0f32126-f0f0-4a25-b4f9-11449b9a6d23"
-      (reference "#PWR?") (unit 1) (value "GND") (footprint "")
-    )
     (path "/db8c5faa-57ff-4d9f-b5e2-863632b44815"
       (reference "#PWR?") (unit 1) (value "GND") (footprint "")
@@
       (reference "#PWR?") (unit 1) (value "GND") (footprint "")
     )
-    (path "/ed6335e6-31ab-4b1c-8195-519d0078ba61"
-      (reference "#PWR?") (unit 1) (value "GND") (footprint "")
-    )
